Commit message: Add files via upload

File: src/wall_climber/urdf/pantograph_arm.xacro (robot description, xacro)
@@ -33,4 +33,7 @@
         <xacro:property name="marker_tip_r"  value="0.006"/>  <!-- marker tip radius        -->
         <xacro:property name="marker_tip_h"  value="0.012"/>  <!-- marker tip length        -->
+        <xacro:property name="marker_tip_contact_r" value="0.004"/> <!-- smooth contact sphere -->
+        <xacro:property name="marker_tip_front_z" value="${-(marker_h + marker_tip_h + 0.002) + 0.03}"/>
+        <xacro:property name="marker_tip_contact_z" value="${marker_tip_front_z + marker_tip_contact_r}"/>
         <xacro:property name="arm_y"         value="0.10"/>   <!-- Y offset on chassis (top edge) -->
         <xacro:property name="arm_z"         value="0"/> <!-- Z offset (wall-facing side) -->
@@ -201,8 +204,10 @@
                 <material name="tip_dark"><color rgba="0.08 0.08 0.08 1.0"/></material>
             </visual>
-            <!-- No collision on marker — trail is drawn in software by
-                 the supervisor.  Removing collision prevents the pen
-                 tip from catching on the whiteboard and tilting the
-                 robot off its 0°/90° driving axes. -->
+            <!-- A small spherical contact tip gives smoother sliding on the board
+                 while keeping the physical contact patch compact and low-catching. -->
+            <collision>
+                <origin xyz="0 0 ${marker_tip_contact_z}"/>
+                <geometry><sphere radius="${marker_tip_contact_r}"/></geometry>
+            </collision>
             <inertial>
                 <origin xyz="0 0 ${-marker_h/2 + 0.03}"/>

Commit message: Add files via upload

File: src/wall_climber/urdf/pantograph_arm.xacro (robot description, xacro)
@@ -180,5 +180,5 @@
             <origin xyz="0 ${fore_len} 0" rpy="0 0 0"/>
             <axis xyz="0 0 1"/>
-            <limit lower="-0.04" upper="0.02" effort="20" velocity="1.2"/>
+            <limit lower="-0.04" upper="0.02" effort="20" velocity="3.0"/>
             <dynamics damping="0.1" friction="0.05"/>
         </joint>
